Commit message: added gripper thing..

File: src/robotic_arm/urdf/robotic_arm.urdf (robot description, URDF)
Before this commit: robot robotic_arm, 4 links, 3 joints
Links:
- added link link5; visual box size=0.12 0.02 0.01
- added link link6; visual box size=0.01 0.016 0.035
- added link link7; visual box size=0.01 0.016 0.035
- link link4: geometry visual mesh filename=package://robotic_arm/mesh/4_.dae scale=10 10 10
Joints:
- added joint link4_link5: type fixed, parent link4, child link5, origin xyz=0 0 0.5 rpy=0 0 0, axis 0 1 0
- added joint link5_link6: type prismatic, parent link5, child link6, origin xyz=-0.008 0 0.02 , axis -1 0 0, limit lower=0.0 upper=0.05 effort=10.0 velocity=0.5
- added joint link5_link7: type prismatic, parent link5, child link7, origin xyz=0.008 0 0.02 , axis 1 0 0, limit lower=0.0 upper=0.05 effort=10.0 velocity=0.5, mimic joint=link5_link6 multiplier=1.0 offset=0.0
